Commit message: a

File: urdf/turtlebot3_waffle_pi.gazebo.xacro (robot description, xacro)
@@ -136,32 +136,33 @@
 <!--link : https://www.raspberrypi.org/documentation/hardware/camera/-->
   <gazebo reference="camera_rgb_frame">
-    <sensor type="camera" name="camera">
-          <pose>0 0 0 0 1.5707 1.5707</pose>
-          <update_rate>30.0</update_rate>
-          <camera name="head">
-            <horizontal_fov>2.0944</horizontal_fov>
-            <image>
-              <width>800</width>
-              <height>800</height>
+    <sensor type="camera" name="Pi Camera">
+      <always_on>true</always_on>
+      <visualize>$(arg camera_visual)</visualize>
+      <camera>
+          <horizontal_fov>1.085595</horizontal_fov>
+          <image>
+              <width>640</width>
+              <height>480</height>
               <format>R8G8B8</format>
-            </image>
-          </camera>
-          <plugin name="camera_plugin" filename="libgazebo_ros_camera.so">
-            <alwaysOn>true</alwaysOn>
-            <updateRate>30.0</updateRate>
-            <cameraName>camera</cameraName>
-            <imageTopicName>image_raw</imageTopicName>
-            <cameraInfoTopicName>camera_info</cameraInfoTopicName>
-            <frameName>camera_link</frameName>
-            <hackBaseline>0.07</hackBaseline>
-            <distortionK1>0.0</distortionK1>
-            <distortionK2>0.0</distortionK2>
-            <distortionK3>0.0</distortionK3>
-            <distortionT1>0.0</distortionT1>
-            <distortionT2>0.0</distortionT2>
-            <robotNamespace></robotNamespace>
-            <tf_prefix_></tf_prefix_>
-          </plugin>
-          <visualize>true</visualize>
+          </image>
+          <clip>
+              <near>0.03</near>
+              <far>100</far>
+          </clip>
+      </camera>
+      <plugin name="camera_controller" filename="libgazebo_ros_camera.so">
+        <alwaysOn>true</alwaysOn>
+        <updateRate>30.0</updateRate>
+        <cameraName>camera</cameraName>
+        <frameName>camera_rgb_optical_frame</frameName>
+        <imageTopicName>rgb/image_raw</imageTopicName>
+        <cameraInfoTopicName>rgb/camera_info</cameraInfoTopicName>
+        <hackBaseline>0.07</hackBaseline>
+        <distortionK1>0.0</distortionK1>
+        <distortionK2>0.0</distortionK2>
+        <distortionK3>0.0</distortionK3>
+        <distortionT1>0.0</distortionT1>
+        <distortionT2>0.0</distortionT2>
+      </plugin>
     </sensor>
   </gazebo>

File: urdf/turtlebot3_waffle_pi.urdf.xacro (robot description, xacro)
@@ -1,24 +1,24 @@
 <?xml version="1.0" ?>
 <robot name="turtlebot3_waffle_pi" xmlns:xacro="http://ros.org/wiki/xacro">
-  <xacro:include filename="$(find aruco_detection)/urdf/common_properties.xacro"/>
-  <xacro:include filename="$(find aruco_detection)/urdf/turtlebot3_waffle_pi.gazebo.xacro"/>
+  <xacro:include filename="$(find turtlebot3_description)/urdf/common_properties.xacro"/>
+  <xacro:include filename="$(find turtlebot3_description)/urdf/turtlebot3_waffle_pi.gazebo.xacro"/>
   <link name="base_footprint"/>
   <joint name="base_joint" type="fixed">
     <parent link="base_footprint"/>
     <child link="base_link" />
-    <origin xyz="0 0 0.005" rpy="0 0 0"/>
+    <origin xyz="0 0 0.010" rpy="0 0 0"/>
   </joint>
   <link name="base_link">
     <visual>
-      <origin xyz="-0.032 0 0.0" rpy="0 0 0"/>
+      <origin xyz="-0.064 0 0.0" rpy="0 0 0"/>
       <geometry>
-        <mesh filename="package://aruco_detection/meshes/bases/waffle_pi_base.stl" scale="0.0005 0.0005 0.0005"/>
+        <mesh filename="package://turtlebot3_description/meshes/bases/waffle_pi_base.stl" scale="0.001 0.001 0.001"/>
       </geometry>
       <material name="light_black"/>
     </visual>
     <collision>
-      <origin xyz="-0.032 0 0.0235" rpy="0 0 0"/>
+      <origin xyz="-0.064 0 0.047" rpy="0 0 0"/>
       <geometry>
-        <box size="0.133 0.133 0.047"/>
+        <box size="0.266 0.266 0.094"/>
       </geometry>
     </collision>
@@ -34,5 +34,5 @@
     <parent link="base_link"/>
     <child link="wheel_left_link"/>
-    <origin xyz="0.0 0.072 0.0050" rpy="-1.57 0 0"/>
+    <origin xyz="0.0 0.144 0.023" rpy="-1.57 0 0"/>
     <axis xyz="0 0 1"/>
   </joint>
@@ -41,5 +41,5 @@
       <origin xyz="0 0 0" rpy="1.57 0 0"/>
       <geometry>
-        <mesh filename="package://aruco_detection/meshes/wheels/left_tire.stl" scale="0.0005 0.0005 0.0005"/>
+        <mesh filename="package://turtlebot3_description/meshes/wheels/left_tire.stl" scale="0.001 0.001 0.001"/>
       </geometry>
       <material name="dark"/>
@@ -48,5 +48,5 @@
       <origin xyz="0 0 0" rpy="0 0 0"/>
       <geometry>
-        <cylinder length="0.009" radius="0.0165"/>
+        <cylinder length="0.018" radius="0.033"/>
       </geometry>
     </collision>
@@ -62,5 +62,5 @@
     <parent link="base_link"/>
     <child link="wheel_right_link"/>
-    <origin xyz="0.0 -0.072 0.0050" rpy="-1.57 0 0"/>
+    <origin xyz="0.0 -0.144 0.023" rpy="-1.57 0 0"/>
     <axis xyz="0 0 1"/>
   </joint>
@@ -69,5 +69,5 @@
       <origin xyz="0 0 0" rpy="1.57 0 0"/>
       <geometry>
-        <mesh filename="package://aruco_detection/meshes/wheels/right_tire.stl" scale="0.0005 0.0005 0.0005"/>
+        <mesh filename="package://turtlebot3_description/meshes/wheels/right_tire.stl" scale="0.001 0.001 0.001"/>
       </geometry>
       <material name="dark"/>
@@ -76,5 +76,5 @@
       <origin xyz="0 0 0" rpy="0 0 0"/>
       <geometry>
-        <cylinder length="0.009" radius="0.0165"/>
+        <cylinder length="0.018" radius="0.033"/>
       </geometry>
     </collision>
@@ -90,16 +90,16 @@
     <parent link="base_link"/>
     <child link="caster_back_right_link"/>
-    <origin xyz="-0.088 -0.032 -0.002" rpy="-1.57 0 0"/>
+    <origin xyz="-0.177 -0.064 -0.004" rpy="-1.57 0 0"/>
   </joint>
   <link name="caster_back_right_link">
     <collision>
-      <origin xyz="0 0.0005 0" rpy="0 0 0"/>
+      <origin xyz="0 0.001 0" rpy="0 0 0"/>
       <geometry>
-        <box size="0.015 0.0045 0.010"/>
+        <box size="0.030 0.009 0.020"/>
       </geometry>
     </collision>
     <inertial>
       <origin xyz="0 0 0" />
-      <mass value="0.0025" />
+      <mass value="0.005" />
       <inertia ixx="0.001" ixy="0.0" ixz="0.0"
                iyy="0.001" iyz="0.0"
@@ -110,16 +110,16 @@
     <parent link="base_link"/>
     <child link="caster_back_left_link"/>
-    <origin xyz="-0.088 0.032 -0.002" rpy="-1.57 0 0"/>
+    <origin xyz="-0.177 0.064 -0.004" rpy="-1.57 0 0"/>
   </joint>
   <link name="caster_back_left_link">
     <collision>
-      <origin xyz="0 0.0005 0" rpy="0 0 0"/>
+      <origin xyz="0 0.001 0" rpy="0 0 0"/>
       <geometry>
-        <box size="0.015 0.0045 0.010"/>
+        <box size="0.030 0.009 0.020"/>
       </geometry>
     </collision>
     <inertial>
       <origin xyz="0 0 0" />
-      <mass value="0.0025" />
+      <mass value="0.005" />
       <inertia ixx="0.001" ixy="0.0" ixz="0.0"
                iyy="0.001" iyz="0.0"
@@ -130,5 +130,5 @@
     <parent link="base_link"/>
     <child link="imu_link"/>
-    <origin xyz="0.0 0 0.034" rpy="0 0 0"/>
+    <origin xyz="0.0 0 0.068" rpy="0 0 0"/>
   </joint>
   <link name="imu_link"/>
@@ -136,5 +136,5 @@
     <parent link="base_link"/>
     <child link="base_scan"/>
-    <origin xyz="-0.020 0 0.061" rpy="0 0 0"/>
+    <origin xyz="-0.064 0 0.122" rpy="0 0 0"/>
   </joint>
   <link name="base_scan">
@@ -142,16 +142,16 @@
       <origin xyz="0 0 0.0" rpy="0 0 0"/>
       <geometry>
-        <mesh filename="package://aruco_detection/meshes/sensors/lds.stl" scale="0.0005 0.0005 0.0005"/>
+        <mesh filename="package://turtlebot3_description/meshes/sensors/lds.stl" scale="0.001 0.001 0.001"/>
       </geometry>
       <material name="dark"/>
     </visual>
     <collision>
-      <origin xyz="0.0075 0 -0.00325" rpy="0 0 0"/>
+      <origin xyz="0.015 0 -0.0065" rpy="0 0 0"/>
       <geometry>
-        <cylinder length="0.0157" radius="0.0275"/>
+        <cylinder length="0.0315" radius="0.055"/>
       </geometry>
     </collision>
     <inertial>
-      <mass value="0.080" />
+      <mass value="0.114" />
       <origin xyz="0 0 0" />
       <inertia ixx="0.001" ixy="0.0" ixz="0.0"
@@ -161,5 +161,5 @@
   </link>
   <joint name="camera_joint" type="fixed">
-    <origin xyz="0.0365 -0.0055 0.042" rpy="0 0 0"/>
+    <origin xyz="0.073 -0.011 0.084" rpy="0 0 0"/>
     <parent link="base_link"/>
     <child link="camera_link"/>
@@ -167,12 +167,12 @@
   <link name="camera_link">
     <collision>
-      <origin xyz="0.0025 0.0055 0.0065" rpy="0 0 0"/>
+      <origin xyz="0.005 0.011 0.013" rpy="0 0 0"/>
       <geometry>
-        <box size="0.0075 0.015 0.0135"/>
+        <box size="0.015 0.030 0.027"/>
       </geometry>
     </collision>
   </link>
   <joint name="camera_rgb_joint" type="fixed">
-    <origin xyz="0.0015 0.0055 0.0045" rpy="0 0 0"/>
+    <origin xyz="0.003 0.011 0.009" rpy="0 0 0"/>
     <parent link="camera_link"/>
     <child link="camera_rgb_frame"/>
